Commit message: Update spot.urdf

File: spot.urdf (robot description, URDF)
Before this commit: robot spot, 25 links, 24 joints
Links:
- removed link base_inertia
- removed link chassis_left
- removed link chassis_right
- added link back_left_lower_CFP, mass 0.005; visual mesh filename=package://mini_ros/stl/OpenQuadruped/LEFT_LOWER_CFP.stl scale=1 1 1
- added link back_left_lower_IMU, mass 0.005; visual mesh filename=package://mini_ros/stl/OpenQuadruped/LEFT_FOOT_IMU.stl scale=1 1 1
- added link back_left_lower_servo, mass 0.005; visual mesh filename=package://mini_ros/stl/OpenQuadruped/LEFT_LOWER_SERVO.stl scale=1 1 1
- added link back_left_upper_CFP, mass 0.005; visual mesh filename=package://mini_ros/stl/OpenQuadruped/LEFT_UPPER_CFP.stl scale=1 1 1
- added link back_left_upper_servo, mass 0.005; visual mesh filename=package://mini_ros/stl/OpenQuadruped/LEFT_UPPER_SERVO.stl scale=1 1 1
- added link back_right_lower_CFP, mass 0.005; visual mesh filename=package://mini_ros/stl/OpenQuadruped/RIGHT_LOWER_CFP.stl scale=1 1 1
- added link back_right_lower_IMU, mass 0.005; visual mesh filename=package://mini_ros/stl/OpenQuadruped/RIGHT_FOOT_IMU.stl scale=1 1 1
- added link back_right_lower_servo, mass 0.005; visual mesh filename=package://mini_ros/stl/OpenQuadruped/RIGHT_LOWER_SERVO.stl scale=1 1 1
- added link back_right_upper_CFP, mass 0.005; visual mesh filename=package://mini_ros/stl/OpenQuadruped/RIGHT_UPPER_CFP.stl scale=1 1 1
- added link back_right_upper_servo, mass 0.005; visual mesh filename=package://mini_ros/stl/OpenQuadruped/RIGHT_UPPER_SERVO.stl scale=1 1 1
- added link cfr_core, mass 0.05; visual mesh filename=package://mini_ros/stl/OpenQuadruped/cfr_core.stl scale=1 1 1
- added link front_left_lower_CFP, mass 0.005; visual mesh filename=package://mini_ros/stl/OpenQuadruped/LEFT_LOWER_CFP.stl scale=1 1 1
- added link front_left_lower_IMU, mass 0.005; visual mesh filename=package://mini_ros/stl/OpenQuadruped/LEFT_FOOT_IMU.stl scale=1 1 1
- added link front_left_lower_servo, mass 0.005; visual mesh filename=package://mini_ros/stl/OpenQuadruped/LEFT_LOWER_SERVO.stl scale=1 1 1
- added link front_left_upper_CFP, mass 0.005; visual mesh filename=package://mini_ros/stl/OpenQuadruped/LEFT_UPPER_CFP.stl scale=1 1 1
- added link front_left_upper_servo, mass 0.005; visual mesh filename=package://mini_ros/stl/OpenQuadruped/LEFT_UPPER_SERVO.stl scale=1 1 1
- added link front_right_lower_CFP, mass 0.005; visual mesh filename=package://mini_ros/stl/OpenQuadruped/RIGHT_LOWER_CFP.stl scale=1 1 1
- added link front_right_lower_IMU, mass 0.005; visual mesh filename=package://mini_ros/stl/OpenQuadruped/RIGHT_FOOT_IMU.stl scale=1 1 1
- added link front_right_lower_servo, mass 0.005; visual mesh filename=package://mini_ros/stl/OpenQuadruped/RIGHT_LOWER_SERVO.stl scale=1 1 1
- added link front_right_upper_CFP, mass 0.005; visual mesh filename=package://mini_ros/stl/OpenQuadruped/RIGHT_UPPER_CFP.stl scale=1 1 1
- added link front_right_upper_servo, mass 0.005; visual mesh filename=package://mini_ros/stl/OpenQuadruped/RIGHT_UPPER_SERVO.stl scale=1 1 1
- added link insta_360, mass 0.5; collision box size=0.03 0.05 0.1; visual mesh filename=package://mini_ros/stl/OpenQuadruped/INSTA360.stl scale=1 1 1
- added link m5paper, mass 0.05; visual mesh filename=package://mini_ros/stl/OpenQuadruped/m5paper.stl scale=1 1 1
- added link oak_d_lite, mass 0.1; visual mesh filename=package://mini_ros/stl/OpenQuadruped/OAKD_LITE.stl scale=1 1 1
- added link rpi_5, mass 0.1; visual mesh filename=package://mini_ros/stl/OpenQuadruped/RPI5.stl scale=1 1 1
- added link rpi_lidar, mass 0.25; collision box size=0.08 0.08 0.05; visual mesh filename=package://mini_ros/stl/OpenQuadruped/lidar.stl scale=1 1 1
- link back: mass 0.1 -> 0.3; geometry collision box size=0.06 0.005 0.06; visual mesh filename=package://mini_ros/stl/OpenQuadruped/m5fire_black.stl scale=1 1 1
- link back_bracket: geometry collision box size=0.1 0.075 0.085; visual mesh filename=package://mini_ros/stl/OpenQuadruped/Back_Bracket.stl scale=1 1 1
- link back_left_lower_leg: geometry collision box size=0.035 0.035 0.11; visual mesh filename=package://mini_ros/stl/OpenQuadruped/LEFT_LOWER_LEG.stl scale=1 1 1
- link back_right_lower_leg: geometry collision box size=0.035 0.035 0.11; visual mesh filename=package://mini_ros/stl/OpenQuadruped/RIGHT_LOWER_LEG.stl scale=1 1 1
- link back_right_upper_leg: geometry collision box size=0.045 0.035 0.11; visual mesh filename=package://mini_ros/stl/OpenQuadruped/RIGHT_UPPER_LEG.stl scale=1 1 1
- link base_link: mass None -> 0.6; geometry collision box size=0.05 0.2 0.08; visual mesh filename=package://mini_ros/stl/OpenQuadruped/MAINBODY.stl scale=1 1 1
- link battery: mass 0.4 -> 1; geometry visual mesh filename=package://mini_ros/stl/OpenQuadruped/Battery.stl scale=1 1 1
- link front_left_lower_leg: geometry collision box size=0.035 0.035 0.11; visual mesh filename=package://mini_ros/stl/OpenQuadruped/LEFT_LOWER_LEG.stl scale=1 1 1
- link front_right_lower_leg: geometry collision box size=0.035 0.035 0.11; visual mesh filename=package://mini_ros/stl/OpenQuadruped/RIGHT_LOWER_LEG.stl scale=1 1 1
Joints:
- removed joint base_base
- removed joint base_left
- removed joint base_right
- added joint back_left_leg_lower_CFP: type fixed, parent back_left_lower_leg, child back_left_lower_CFP, origin xyz=0 0 0 rpy=0 0 0
- added joint back_left_leg_lower_IMU: type fixed, parent back_left_lower_leg, child back_left_lower_IMU, origin xyz=0 0 0 rpy=0 0 0
- added joint back_left_leg_lower_servo: type fixed, parent back_left_lower_leg, child back_left_lower_servo, origin xyz=0 0 0 rpy=0 0 0
- added joint back_left_leg_upper_CFP: type fixed, parent back_left_upper_leg, child back_left_upper_CFP, origin xyz=0 0 0 rpy=0 0 0
- added joint back_left_leg_upper_servo: type fixed, parent back_left_upper_leg, child back_left_upper_servo, origin xyz=0 0 0 rpy=0 0 0
- added joint back_right_leg_lower_CFP: type fixed, parent back_right_lower_leg, child back_right_lower_CFP, origin xyz=0 0 -0.1265 rpy=0 0 0
- added joint back_right_leg_lower_IMU: type fixed, parent back_right_lower_leg, child back_right_lower_IMU, origin xyz=0 0 -0.1265 rpy=0 0 0
- added joint back_right_leg_lower_servo: type fixed, parent back_right_lower_leg, child back_right_lower_servo, origin xyz=0 0 -0.1265 rpy=0 0 0
- added joint back_right_leg_upper_CFP: type fixed, parent back_right_upper_leg, child back_right_upper_CFP, origin xyz=0 0 0 rpy=0 0 0
- added joint back_right_leg_upper_servo: type fixed, parent back_right_upper_leg, child back_right_upper_servo, origin xyz=0 0 0 rpy=0 0 0
- added joint base_cfr_core: type fixed, parent base_link, child cfr_core, origin xyz=-0.01 0 -0.0225 rpy=0 0 0
- added joint base_insta360: type fixed, parent base_link, child insta_360, origin xyz=-0.01 0 -0.0225 rpy=0 0 0
- added joint base_m5paper: type fixed, parent base_link, child m5paper, origin xyz=-0.01 0 -0.0225 rpy=0 0 0
- added joint base_oakd_lite: type fixed, parent base_link, child oak_d_lite, origin xyz=-0.01 0 -0.0225 rpy=0 0 0
- added joint base_rpi_5: type fixed, parent base_link, child rpi_5, origin xyz=-0.01 0 -0.0225 rpy=0 0 0
- added joint base_rpi_lidar: type fixed, parent base_link, child rpi_lidar, origin xyz=-0.01 0 -0.0225 rpy=0 0 0
- added joint front_left_leg_lower_CFP: type fixed, parent front_left_lower_leg, child front_left_lower_CFP, origin xyz=0 0 0 rpy=0 0 0
- added joint front_left_leg_lower_IMU: type fixed, parent front_left_lower_leg, child front_left_lower_IMU, origin xyz=0 0 0 rpy=0 0 0
- added joint front_left_leg_lower_servo: type fixed, parent front_left_lower_leg, child front_left_lower_servo, origin xyz=0 0 0 rpy=0 0 0
- added joint front_left_leg_upper_CFP: type fixed, parent front_left_upper_leg, child front_left_upper_CFP, origin xyz=0 0 0 rpy=0 0 0
- added joint front_left_leg_upper_servo: type fixed, parent front_left_upper_leg, child front_left_upper_servo, origin xyz=0 0 0 rpy=0 0 0
- added joint front_right_leg_lower_CFP: type fixed, parent front_right_lower_leg, child front_right_lower_CFP, origin xyz=0 0 -0.1265 rpy=0 0 0
- added joint front_right_leg_lower_IMU: type fixed, parent front_right_lower_leg, child front_right_lower_IMU, origin xyz=0 0 -0.1265 rpy=0 0 0
- added joint front_right_leg_lower_servo: type fixed, parent front_right_lower_leg, child front_right_lower_servo, origin xyz=0 0 -0.1265 rpy=0 0 0
- added joint front_right_leg_upper_CFP: type fixed, parent front_right_upper_leg, child front_right_upper_CFP, origin xyz=0 0 0 rpy=0 0 0
- added joint front_right_leg_upper_servo: type fixed, parent front_right_upper_leg, child front_right_upper_servo, origin xyz=0 0 0 rpy=0 0 0
- joint back_right_leg_foot: origin xyz=0 0 -0.1265 rpy=0 0 0 -> xyz=0 0 -0.1 rpy=0 0 0
- joint front_right_leg_foot: origin xyz=0 0 -0.1265 rpy=0 0 0 -> xyz=0 0 -0.1 rpy=0 0 0
- joint motor_back_left_hip: origin xyz=-0.1365 0.0394 0.022 rpy=0 0 0 -> xyz=-0.1075 0.0394 0.017 rpy=0 0 0
- joint motor_back_left_lower_leg: origin xyz=-0.005 0.018 -0.109 rpy=0 0 0 -> xyz=-0.005 0.002 -0.1068 rpy=0 0 0
- joint motor_back_left_upper_leg: origin xyz=0.0015 0.045 -0.0087 rpy=0 0 0 -> xyz=0.0015 0.045 -0.011 rpy=0 0 0
- joint motor_back_right_hip: origin xyz=-0.1365 -0.0394 0.022 rpy=0 0 0 -> xyz=-0.1075 -0.0394 0.017 rpy=0 0 0
- joint motor_back_right_lower_leg: origin xyz=-0.005 -0.018 -0.109 rpy=0 0 0 -> xyz=-0.005 -0.002 -0.1068 rpy=0 0 0
- joint motor_back_right_upper_leg: origin xyz=0.0015 -0.045 -0.0087 rpy=0 0 0 -> xyz=0.0015 -0.045 -0.011 rpy=0 0 0
- joint motor_front_left_hip: origin xyz=0.0915 0.0394 0.022 rpy=0 0 0 -> xyz=0.0995 0.0394 0.017 rpy=0 0 0
- joint motor_front_left_lower_leg: origin xyz=-0.005 0.018 -0.109 rpy=0 0 0 -> xyz=-0.005 0.002 -0.1068 rpy=0 0 0
- joint motor_front_left_upper_leg: origin xyz=0.0015 0.045 -0.0087 rpy=0 0 0 -> xyz=0.0015 0.045 -0.011 rpy=0 0 0
- joint motor_front_right_hip: origin xyz=0.0915 -0.0394 0.022 rpy=0 0 0 -> xyz=0.0995 -0.0394 0.017 rpy=0 0 0
- joint motor_front_right_lower_leg: origin xyz=-0.005 -0.018 -0.109 rpy=0 0 0 -> xyz=-0.005 -0.002 -0.1068 rpy=0 0 0
- joint motor_front_right_upper_leg: origin xyz=0.0015 -0.045 -0.0087 rpy=0 0 0 -> xyz=0.0015 -0.045 -0.011 rpy=0 0 0
